File: proyecto_v2/proyecto_v2.kicad_sch (KiCad schematic)
At the start: 38 parts, among them J1 Sensor Inductivo, J10 esp32, J11 ENTRADA, J2 Servo, J3 Sensor Óptico, J4 Sensor Ultrasónico, J5 Sensor Capacitivo, J6 Final Carrera 1, J7 Final Carrera 2, J8 Final Carrera 3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

Commit message: schematic
Parts:
- added J?: Display LCD, symbol Connector:Conn_01x04_Male
Connections:
- net +12V: now also J?.2 (Pin_2)
- net GND: now also J?.1 (Pin_1)
- net PIN 19: now reaches J9.12 (Pin_12)
- net PIN 21: now reaches J9.14 (Pin_14)
- net PIN 21: now also J?.3 (Pin_3)
- net PIN 22: now reaches J9.17 (Pin_17)
- net PIN 22: now also J?.4 (Pin_4)
- net PIN 23: now reaches J9.18 (Pin_18)
Changed lines of the file:
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@@
+    (stroke (width 0) (type default) (color 0 0 0 0))
+  )
+  (wire (pts (xy 220.98 59.69) (xy 227.33 59.69))
     (stroke (width 0) (type default) (color 0 0 0 0))
   )
@@
     (stroke (width 0) (type default) (color 0 0 0 0))
   )
+  (wire (pts (xy 220.98 54.61) (xy 227.33 54.61))
+    (stroke (width 0) (type default) (color 0 0 0 0))
+  )
   (wire (pts (xy 36.83 35.56) (xy 49.53 35.56))
     (stroke (width 0) (type default) (color 0 0 0 0))
@@
     (stroke (width 0) (type default) (color 0 0 0 0))
   )
+  (wire (pts (xy 215.9 97.79) (xy 220.98 97.79))
+    (stroke (width 0) (type default) (color 0 0 0 0))
+  )
   (wire (pts (xy 240.03 52.07) (xy 247.65 52.07))
     (stroke (width 0) (type default) (color 0 0 0 0))
@@
     (stroke (width 0) (type default) (color 0 0 0 0))
   )
+  (wire (pts (xy 219.71 69.85) (xy 227.33 69.85))
+    (stroke (width 0) (type default) (color 0 0 0 0))
+  )
   (wire (pts (xy 121.92 46.99) (xy 127 46.99))
     (stroke (width 0) (type default) (color 0 0 0 0))
   )
+  (wire (pts (xy 215.9 95.25) (xy 220.98 95.25))
+    (stroke (width 0) (type default) (color 0 0 0 0))
+  )
   (wire (pts (xy 240.03 39.37) (xy 243.84 39.37))
     (stroke (width 0) (type default) (color 0 0 0 0))
@@
     (stroke (width 0) (type default) (color 0 0 0 0))
   )
+  (wire (pts (xy 215.9 100.33) (xy 223.52 100.33))
+    (stroke (width 0) (type default) (color 0 0 0 0))
+  )
   (wire (pts (xy 121.92 52.07) (xy 127 52.07))
     (stroke (width 0) (type default) (color 0 0 0 0))
@@
     (stroke (width 0) (type default) (color 0 0 0 0))
   )
+  (wire (pts (xy 215.9 102.87) (xy 223.52 102.87))
+    (stroke (width 0) (type default) (color 0 0 0 0))
+  )
   (wire (pts (xy 46.99 125.73) (xy 46.99 129.54))
     (stroke (width 0) (type default) (color 0 0 0 0))
@@
   )
   (wire (pts (xy 71.12 127) (xy 71.12 130.81))
+    (stroke (width 0) (type default) (color 0 0 0 0))
+  )
+  (wire (pts (xy 219.71 67.31) (xy 227.33 67.31))
     (stroke (width 0) (type default) (color 0 0 0 0))
   )
@@
     (effects (font (size 1.27 1.27)) (justify left bottom))
   )
+  (label "PIN 19" (at 220.98 54.61 180)
+    (effects (font (size 1.27 1.27)) (justify right bottom))
+  )
   (label "PIN 27" (at 52.07 172.72 180)
     (effects (font (size 1.27 1.27)) (justify right bottom))
@@
     (effects (font (size 1.27 1.27)) (justify left bottom))
   )
+  (label "PIN 22" (at 223.52 102.87 0)
+    (effects (font (size 1.27 1.27)) (justify left bottom))
+  )
+  (label "PIN 22" (at 219.71 67.31 180)
+    (effects (font (size 1.27 1.27)) (justify right bottom))
+  )
   (label "PIN 25" (at 58.42 138.43 180)
     (effects (font (size 1.27 1.27)) (justify right bottom))
@@
     (effects (font (size 1.27 1.27)) (justify left bottom))
   )
+  (label "PIN 21" (at 220.98 59.69 180)
+    (effects (font (size 1.27 1.27)) (justify right bottom))
+  )
   (label "FC3" (at 158.75 63.5 0)
     (effects (font (size 1.27 1.27)) (justify left bottom))
@@
     (effects (font (size 1.27 1.27)) (justify left bottom))
   )
+  (label "PIN 23" (at 219.71 69.85 180)
+    (effects (font (size 1.27 1.27)) (justify right bottom))
+  )
   (label "FC1" (at 158.75 38.1 0)
     (effects (font (size 1.27 1.27)) (justify left bottom))
@@
   )
   (label "PIN 27" (at 247.65 46.99 0)
+    (effects (font (size 1.27 1.27)) (justify left bottom))
+  )
+  (label "PIN 21" (at 223.52 100.33 0)
     (effects (font (size 1.27 1.27)) (justify left bottom))
   )
@@
     )
     (pin "1")
+  )
+  (symbol (lib_id "Connector:Conn_01x04_Male") (at 210.82 97.79 0) (unit 1)
+    (in_bom yes) (on_board yes) (fields_autoplaced)
+    (property "Reference" "J?" (id 0) (at 211.455 90.17 0))
+    (property "Value" "Display LCD" (id 1) (at 211.455 92.71 0))
+    (property "Footprint" "" (id 2) (at 210.82 97.79 0)
+      (effects (font (size 1.27 1.27)) hide)
+    )
+    (property "Datasheet" "~" (id 3) (at 210.82 97.79 0)
+      (effects (font (size 1.27 1.27)) hide)
+    )
+    (pin "1")
+    (pin "2")
+    (pin "3")
+    (pin "4")
   )
   (symbol (lib_id "Connector:Conn_01x19_Male") (at 234.95 49.53 0) (unit 1)
@@
     (pin "1")
   )
+  (symbol (lib_id "power:+12V") (at 220.98 97.79 270) (unit 1)
+    (in_bom yes) (on_board yes) (fields_autoplaced)
+    (property "Reference" "#PWR?" (id 0) (at 217.17 97.79 0)
+      (effects (font (size 1.27 1.27)) hide)
+    )
+    (property "Value" "+12V" (id 1) (at 224.79 97.7899 90)
+      (effects (font (size 1.27 1.27)) (justify left))
+    )
+    (property "Footprint" "" (id 2) (at 220.98 97.79 0)
+      (effects (font (size 1.27 1.27)) hide)
+    )
+    (property "Datasheet" "" (id 3) (at 220.98 97.79 0)
+      (effects (font (size 1.27 1.27)) hide)
+    )
+    (pin "1")
+  )
   (symbol (lib_id "power:GND") (at 36.83 38.1 0) (unit 1)
     (in_bom yes) (on_board yes) (fields_autoplaced)
@@
     (pin "1")
     (pin "2")
+  )
+  (symbol (lib_id "power:GND") (at 220.98 95.25 90) (unit 1)
+    (in_bom yes) (on_board yes) (fields_autoplaced)
+    (property "Reference" "#PWR?" (id 0) (at 227.33 95.25 0)
+      (effects (font (size 1.27 1.27)) hide)
+    )
+    (property "Value" "GND" (id 1) (at 224.79 95.2499 90)
+      (effects (font (size 1.27 1.27)) (justify right))
+    )
+    (property "Footprint" "" (id 2) (at 220.98 95.25 0)
+      (effects (font (size 1.27 1.27)) hide)
+    )
+    (property "Datasheet" "" (id 3) (at 220.98 95.25 0)
+      (effects (font (size 1.27 1.27)) hide)
+    )
+    (pin "1")
   )
   (symbol (lib_id "power:+5V") (at 46.99 125.73 0) (unit 1)
@@
       (reference "#PWR0102") (unit 1) (value "GND") (footprint "")
     )
+    (path "/ce684910-884b-4336-abe0-5da59a3241ad"
+      (reference "#PWR?") (unit 1) (value "+12V") (footprint "")
+    )
+    (path "/da7ecff7-8850-4574-a623-de1c6a48340d"
+      (reference "#PWR?") (unit 1) (value "GND") (footprint "")
+    )
     (path "/30287200-a957-4f1e-a743-d8ba13793ebb"
       (reference "C1") (unit 1) (value "0.33uF") (footprint "Capacitor_THT:C_Disc_D3.0mm_W2.0mm_P2.50mm")
@@
       (reference "J11") (unit 1) (value "ENTRADA") (footprint "Connector_PinSocket_1.00mm:PinSocket_1x02_P1.00mm_Vertical")
     )
+    (path "/7855a5bd-7b06-4ceb-b835-3691f7ec2462"
+      (reference "J?") (unit 1) (value "Display LCD") (footprint "")
+    )
     (path "/4ed24e8c-7f2e-4988-a88e-abdd7f867590"
